Commit message: adding a virtual TCP joint for planning

File: src/ur10e_config/robot_description/urdf/ur10e_rg2.urdf (robot description, URDF)
Before this commit: robot ur10e_rg2, 18 links, 17 joints
Links:
- added link arm_tcp_link
Joints:
- added joint arm_tcp_joint: type fixed, parent arm_tool0, child arm_tcp_link, origin xyz=0 -21.5 0 rpy=0 0 0

File: src/ur10e_config/robot_description/urdf/ur10e_rg2.xacro (robot description, xacro)
@@ -18,4 +18,12 @@
       <!-- No origin, using the default all-zero -->
    </joint>
+   <!-- Define a virtual link as the tip link for navigation -->
+   <!-- This is roughly about 21.5cm off from tool0 -->
+   <link name="arm_tcp_link"/>
+   <joint name="arm_tcp_joint" type="fixed">
+      <parent link="arm_tool0"/>
+      <child link="arm_tcp_link"/>
+      <origin xyz="0 -21.5 0" rpy="0 0 0"/>
+   </joint>
    <!-- The world joint will be declared within the moveit package. -->
 </robot>

File: src/ur10e_config/robot_moveit/config/gazebo_ur10e_rg2.urdf (robot description, URDF)
Before this commit: robot ur10e_rg2, 18 links, 17 joints
Links:
- added link arm_tcp_link
Joints:
- added joint arm_tcp_joint: type fixed, parent arm_tool0, child arm_tcp_link, origin xyz=0 -21.5 0 rpy=0 0 0

Commit message: accidentally make the robot virtual target link 21m away from the robot

File: src/ur10e_config/robot_description/urdf/ur10e_rg2.urdf (robot description, URDF)
Before this commit: robot ur10e_rg2, 19 links, 18 joints
Joints:
- joint arm_tcp_joint: origin xyz=0 -21.5 0 rpy=0 0 0 -> xyz=0 0 0.215 rpy=0 0 0

File: src/ur10e_config/robot_description/urdf/ur10e_rg2.xacro (robot description, xacro)
@@ -24,5 +24,5 @@
       <parent link="arm_tool0"/>
       <child link="arm_tcp_link"/>
-      <origin xyz="0 -21.5 0" rpy="0 0 0"/>
+      <origin xyz="0 0 0.215" rpy="0 0 0"/>
    </joint>
    <!-- The world joint will be declared within the moveit package. -->
